File: electronics/ms-pcb/ms-pcb.kicad_sch (KiCad schematic)
At the start: 4 parts

Commit message: elec: first PCB schematic draft
Parts:
- removed J? (x2): BM06B-SRSS-TB_LF__SN_, BM06B-SRSS-TB_LF__SN_:JST_BM06B-SRSS-TB_LF__SN_, symbol JST_SH_6pins:BM06B-SRSS-TB_LF__SN_
- removed U?: ESP32-DEVKITC-32U, ESP32-DEVKITC-32U:MODULE_ESP32-DEVKITC-32U, symbol ESP32-DEVKITC-32U:ESP32-DEVKITC-32U
- added D?: LED_VBAT, symbol Device:LED
- added D?: LED_3V3, symbol Device:LED
- added DRV?: DRV8833, symbol DRV8833:Dual motor driver
- added J?: Right motor, BM06B-SRSS-TB_LF__SN_:JST_BM06B-SRSS-TB_LF__SN_, symbol JST_SH_6pins:BM06B-SRSS-TB_LF__SN_
- added J?: Left motor, BM06B-SRSS-TB_LF__SN_:JST_BM06B-SRSS-TB_LF__SN_, symbol JST_SH_6pins:BM06B-SRSS-TB_LF__SN_
- added LS?: PKLCS1212E20A0-R1, PKLCS1212E20A0-R1:SPKR_PKLCS1212E20A0-R1, symbol PKLCS1212E20A0-R1:PKLCS1212E20A0-R1
- added R? (x2): 220, symbol Device:R
- added R?: 10k, symbol Device:R
- added R?: 1k, symbol Device:R
- added U?: GY-521, GY-521:GY-521, symbol GY-521:GY-521
- added U?: ESP32-S3-DEVKITC-1U-N8R2, ESP32-S3-DEVKITC-1U-N8R2:XCVR_ESP32-S3-DEVKITC-1U-N8R2, symbol ESP32-S3-DEVKITC-1U-N8R2:ESP32-S3-DEVKITC-1U-N8R2
- added VL53L1X? (x5): ToF distance sensor, symbol VL53L1x:ToF distance sensor
Connections:
- net GND: now reaches J?.N (NEG)
- net GND: now also D?.1 (K), D?.1 (K), DRV?.1 (GND), DRV?.15 (AISEN), DRV?.16 (BISEN), DRV?.9 (GND), J?.1 (GND), J?.1 (GND), LS?.N, R?.2, U?.GND, U?.J1_22 (GND), U?.J3_1 (GND), U?.J3_21 (GND), U?.J3_22 (GND), VL53L1X?.2 (GND), VL53L1X?.2 (GND), VL53L1X?.2 (GND), VL53L1X?.2 (GND), VL53L1X?.2 (GND)
- net +BATT: now reaches J?.P (POS)
- net +BATT: now also DRV?.10 (VIN), R?.1, R?.1, R?.1, U?.J1_21 (5V0)
- new net: D?.2 (A), R?.2 (x2)
- new net: J?.S1 (SHIELD), J?.S2 (SHIELD) (x2)
- new net +3.3V: J?.4 (VCC), J?.4 (VCC), U?.J1_1 (3V3), U?.J1_2 (3V3), U?.VCC, VL53L1X?.1 (VIN), VL53L1X?.1 (VIN), VL53L1X?.1 (VIN), VL53L1X?.1 (VIN), VL53L1X?.1 (VIN)
- new net DRV_L1: DRV?.3 (BIN1), U?.J1_8 (GPIO15)
- new net DRV_L2: DRV?.4 (BIN2), U?.J1_9 (GPIO16)
- new net DRV_R1: DRV?.6 (AIN1), U?.J1_10 (GPIO17)
- new net DRV_R2: DRV?.5 (AIN2), U?.J1_11 (GPIO18)
- new net ENC_L1: J?.3 (OUT_A), U?.J1_4 (GPIO4)
- new net ENC_L2: J?.2 (OUT_B), U?.J1_5 (GPIO5)
- new net ENC_R1: J?.3 (OUT_A), U?.J1_6 (GPIO6)
- new net ENC_R2: J?.2 (OUT_B), U?.J1_7 (GPIO7)
- new net MOT_L1: DRV?.11 (BOUT1), J?.6 (M1)
- new net MOT_L2: DRV?.12 (BOUT2), J?.5 (M2)
- new net MOT_R1: DRV?.14 (AOUT1), J?.6 (M1)
- new net MOT_R2: DRV?.13 (AOUT2), J?.5 (M2)
- new net SCL: U?.J3_5 (GPIO2), U?.SCL, VL53L1X?.3 (SCL), VL53L1X?.3 (SCL), VL53L1X?.3 (SCL), VL53L1X?.3 (SCL), VL53L1X?.3 (SCL)
- new net SDA: U?.J3_4 (GPIO1), U?.SDA, VL53L1X?.4 (SDA), VL53L1X?.4 (SDA), VL53L1X?.4 (SDA), VL53L1X?.4 (SDA), VL53L1X?.4 (SDA)
- new net Vmes: R?.1, R?.2
- new net XSHUT_F: U?.J3_8 (MTDO/GPIO40), VL53L1X?.6 (XSHUT)
- new net XSHUT_FL: U?.J3_7 (MTDI/GPIO41), VL53L1X?.6 (XSHUT)
- new net XSHUT_FR: U?.J3_9 (MTCK/GPIO39), VL53L1X?.6 (XSHUT)
- new net XSHUT_L: U?.J3_6 (MTMS/GPIO42), VL53L1X?.6 (XSHUT)
- new net XSHUT_R: U?.J3_10 (GPIO38), VL53L1X?.6 (XSHUT)
- new net buzzer: LS?.P, U?.J1_13 (GPIO3)
- no-connect marks 0 -> 14
Other:
- title: Micromouse PCB -> Algernon Micromouse PCB
- moved on the sheet: J?
