File: electronics/ms-pcb/_autosave-ms-pcb.kicad_sch (KiCad schematic)
At the start: 20 parts, among them J1 Left motor, J2 Right motor, J3 XT60-M, U1 ESP32-S3-DEVKITC-1U-N8R2, U2 GY-521

Commit message: elec: design some missing footprints
Parts:
- D1, D2: footprint (none) -> LED_SMD:LED_1206_3216Metric_Pad1.42x1.75mm_HandSolder
- J1, J2: footprint BM06B-SRSS-TB_LF__SN_:JST_BM06B-SRSS-TB_LF__SN_ -> footprints:JST_SH_6pins
- J3: footprint XT60-M:AMASS_XT60-M -> footprints:AMASS_XT60-M
- LS1: footprint PKLCS1212E20A0-R1:SPKR_PKLCS1212E20A0-R1 -> footprints:SPKR_PKLCS1212E20A0-R1
- R1, R2, R3, R4, R5: footprint (none) -> Resistor_SMD:R_1206_3216Metric_Pad1.30x1.75mm_HandSolder
- VL53L1X1, VL53L1X2, VL53L1X3, VL53L1X4, VL53L1X5: footprint (none) -> Connector_PinHeader_2.54mm:PinHeader_1x06_P2.54mm_Horizontal
Changed lines of the file:
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@@
       (effects (font (size 1.27 1.27)) (justify left))
     )
-    (property "Footprint" "" (id 2) (at 138.43 64.77 0)
+    (property "Footprint" "Connector_PinHeader_2.54mm:PinHeader_1x06_P2.54mm_Horizontal" (id 2) (at 138.43 64.77 0)
       (effects (font (size 1.27 1.27)) hide)
     )
@@
       (effects (font (size 1.27 1.27)) (justify left))
     )
-    (property "Footprint" "" (id 2) (at 191.77 40.64 0)
+    (property "Footprint" "Connector_PinHeader_2.54mm:PinHeader_1x06_P2.54mm_Horizontal" (id 2) (at 191.77 40.64 0)
       (effects (font (size 1.27 1.27)) hide)
     )
@@
       (effects (font (size 1.27 1.27)) (justify left))
     )
-    (property "Footprint" "" (id 2) (at 49.022 165.1 90)
+    (property "Footprint" "Resistor_SMD:R_1206_3216Metric_Pad1.30x1.75mm_HandSolder" (id 2) (at 49.022 165.1 90)
       (effects (font (size 1.27 1.27)) hide)
     )
@@
       (effects (font (size 1.27 1.27)) (justify left))
     )
-    (property "Footprint" "BM06B-SRSS-TB_LF__SN_:JST_BM06B-SRSS-TB_LF__SN_" (id 2) (at 266.7 60.96 0)
+    (property "Footprint" "footprints:JST_SH_6pins" (id 2) (at 266.7 60.96 0)
       (effects (font (size 1.27 1.27)) (justify bottom) hide)
     )
@@
       (effects (font (size 1.27 1.27)) (justify right))
     )
-    (property "Footprint" "" (id 2) (at 33.02 176.53 0)
+    (property "Footprint" "LED_SMD:LED_1206_3216Metric_Pad1.42x1.75mm_HandSolder" (id 2) (at 33.02 176.53 0)
       (effects (font (size 1.27 1.27)) hide)
     )
@@
       (effects (font (size 1.27 1.27)) (justify left))
     )
-    (property "Footprint" "" (id 2) (at 31.242 165.1 90)
+    (property "Footprint" "Resistor_SMD:R_1206_3216Metric_Pad1.30x1.75mm_HandSolder" (id 2) (at 31.242 165.1 90)
       (effects (font (size 1.27 1.27)) hide)
     )
@@
   (symbol (lib_id "power:GND") (at 130.81 144.78 0) (unit 1)
     (in_bom yes) (on_board yes) (fields_autoplaced)
-    (property "Reference" "#PWR?" (id 0) (at 130.81 151.13 0)
+    (property "Reference" "#PWR0101" (id 0) (at 130.81 151.13 0)
       (effects (font (size 1.27 1.27)) hide)
     )
@@
       (effects (font (size 1.27 1.27)) (justify left))
     )
-    (property "Footprint" "" (id 2) (at 66.802 163.83 90)
+    (property "Footprint" "Resistor_SMD:R_1206_3216Metric_Pad1.30x1.75mm_HandSolder" (id 2) (at 66.802 163.83 90)
       (effects (font (size 1.27 1.27)) hide)
     )
@@
       (effects (font (size 1.27 1.27)) (justify left))
     )
-    (property "Footprint" "BM06B-SRSS-TB_LF__SN_:JST_BM06B-SRSS-TB_LF__SN_" (id 2) (at 266.7 29.21 0)
+    (property "Footprint" "footprints:JST_SH_6pins" (id 2) (at 266.7 29.21 0)
       (effects (font (size 1.27 1.27)) (justify bottom) hide)
     )
@@
       (effects (font (size 1.27 1.27)) (justify left))
     )
-    (property "Footprint" "" (id 2) (at 66.802 176.53 90)
+    (property "Footprint" "Resistor_SMD:R_1206_3216Metric_Pad1.30x1.75mm_HandSolder" (id 2) (at 66.802 176.53 90)
       (effects (font (size 1.27 1.27)) hide)
     )
@@
       (effects (font (size 1.27 1.27)) (justify left))
     )
-    (property "Footprint" "" (id 2) (at 191.77 64.77 0)
+    (property "Footprint" "Connector_PinHeader_2.54mm:PinHeader_1x06_P2.54mm_Horizontal" (id 2) (at 191.77 64.77 0)
       (effects (font (size 1.27 1.27)) hide)
     )
@@
       (effects (font (size 1.27 1.27)) (justify left))
     )
-    (property "Footprint" "XT60-M:AMASS_XT60-M" (id 2) (at 39.37 133.35 0)
+    (property "Footprint" "footprints:AMASS_XT60-M" (id 2) (at 39.37 133.35 0)
       (effects (font (size 1.27 1.27)) (justify bottom) hide)
     )
@@
       (effects (font (size 1.27 1.27)) (justify right))
     )
-    (property "Footprint" "" (id 2) (at 50.8 176.53 0)
+    (property "Footprint" "LED_SMD:LED_1206_3216Metric_Pad1.42x1.75mm_HandSolder" (id 2) (at 50.8 176.53 0)
       (effects (font (size 1.27 1.27)) hide)
     )
@@
       (effects (font (size 1.27 1.27)) (justify left))
     )
-    (property "Footprint" "PKLCS1212E20A0-R1:SPKR_PKLCS1212E20A0-R1" (id 2) (at 81.28 134.62 0)
+    (property "Footprint" "footprints:SPKR_PKLCS1212E20A0-R1" (id 2) (at 81.28 134.62 0)
       (effects (font (size 1.27 1.27)) (justify bottom) hide)
     )
@@
       (effects (font (size 1.27 1.27)) (justify left))
     )
-    (property "Footprint" "" (id 2) (at 138.43 88.9 0)
+    (property "Footprint" "Connector_PinHeader_2.54mm:PinHeader_1x06_P2.54mm_Horizontal" (id 2) (at 138.43 88.9 0)
       (effects (font (size 1.27 1.27)) hide)
     )
@@
       (effects (font (size 1.27 1.27)) (justify left))
     )
-    (property "Footprint" "" (id 2) (at 138.43 40.64 0)
+    (property "Footprint" "Connector_PinHeader_2.54mm:PinHeader_1x06_P2.54mm_Horizontal" (id 2) (at 138.43 40.64 0)
       (effects (font (size 1.27 1.27)) hide)
     )
@@
       (effects (font (size 1.27 1.27)) (justify left))
     )
-    (property "Footprint" "" (id 2) (at 113.792 142.24 90)
+    (property "Footprint" "Resistor_SMD:R_1206_3216Metric_Pad1.30x1.75mm_HandSolder" (id 2) (at 113.792 142.24 90)
       (effects (font (size 1.27 1.27)) hide)
     )
@@
     )
     (path "/6d3abdea-bfa7-473c-8a0e-b74a8765736e"
-      (reference "#PWR?") (unit 1) (value "GND") (footprint "")
+      (reference "#PWR0101") (unit 1) (value "GND") (footprint "")
     )
     (path "/640f477c-349e-4544-8313-0567779ba460"
-      (reference "D1") (unit 1) (value "LED_VBAT") (footprint "")
+      (reference "D1") (unit 1) (value "LED_VBAT") (footprint "LED_SMD:LED_1206_3216Metric_Pad1.42x1.75mm_HandSolder")
     )
     (path "/a8246948-cefe-4cb5-800c-1ab5595424cf"
-      (reference "D2") (unit 1) (value "LED_3V3") (footprint "")
+      (reference "D2") (unit 1) (value "LED_3V3") (footprint "LED_SMD:LED_1206_3216Metric_Pad1.42x1.75mm_HandSolder")
     )
     (path "/8a807ff6-0a61-4154-9000-caf05d86c07b"
@@
     )
     (path "/72aa56fc-a28b-4d91-8c02-810f2d6f30cd"
-      (reference "J1") (unit 1) (value "Left motor") (footprint "BM06B-SRSS-TB_LF__SN_:JST_BM06B-SRSS-TB_LF__SN_")
+      (reference "J1") (unit 1) (value "Left motor") (footprint "footprints:JST_SH_6pins")
     )
     (path "/53c61da3-5ed9-4d59-8211-37a02b443a19"
-      (reference "J2") (unit 1) (value "Right motor") (footprint "BM06B-SRSS-TB_LF__SN_:JST_BM06B-SRSS-TB_LF__SN_")
+      (reference "J2") (unit 1) (value "Right motor") (footprint "footprints:JST_SH_6pins")
     )
     (path "/9a32b10d-dbd5-4b1a-ba9f-cad46ec3e360"
-      (reference "J3") (unit 1) (value "XT60-M") (footprint "XT60-M:AMASS_XT60-M")
+      (reference "J3") (unit 1) (value "XT60-M") (footprint "footprints:AMASS_XT60-M")
     )
     (path "/cfea8ce7-c309-415e-ad9d-692c4d19c36e"
-      (reference "LS1") (unit 1) (value "PKLCS1212E20A0-R1") (footprint "PKLCS1212E20A0-R1:SPKR_PKLCS1212E20A0-R1")
+      (reference "LS1") (unit 1) (value "PKLCS1212E20A0-R1") (footprint "footprints:SPKR_PKLCS1212E20A0-R1")
     )
     (path "/f1891062-a12e-4348-907a-d381c1fa2eb1"
-      (reference "R1") (unit 1) (value "100k") (footprint "")
+      (reference "R1") (unit 1) (value "100k") (footprint "Resistor_SMD:R_1206_3216Metric_Pad1.30x1.75mm_HandSolder")
     )
     (path "/71866ac7-d316-405b-bca6-883268e47363"
-      (reference "R2") (unit 1) (value "10k") (footprint "")
+      (reference "R2") (unit 1) (value "10k") (footprint "Resistor_SMD:R_1206_3216Metric_Pad1.30x1.75mm_HandSolder")
     )
     (path "/69312bab-5d49-49ca-81b4-8b6c5ee66692"
-      (reference "R3") (unit 1) (value "220") (footprint "")
+      (reference "R3") (unit 1) (value "220") (footprint "Resistor_SMD:R_1206_3216Metric_Pad1.30x1.75mm_HandSolder")
     )
     (path "/3220fdb9-f086-4442-8abf-51c020752183"
-      (reference "R4") (unit 1) (value "220") (footprint "")
+      (reference "R4") (unit 1) (value "220") (footprint "Resistor_SMD:R_1206_3216Metric_Pad1.30x1.75mm_HandSolder")
     )
     (path "/7dfe908f-2a26-476c-9390-b6c5ecff871d"
-      (reference "R5") (unit 1) (value "1k") (footprint "")
+      (reference "R5") (unit 1) (value "1k") (footprint "Resistor_SMD:R_1206_3216Metric_Pad1.30x1.75mm_HandSolder")
     )
     (path "/b7364b23-2df2-472a-8caa-f6c5aa8ed4c7"
@@
     )
     (path "/db5a9986-4aac-4288-bd76-d31395dc1fc5"
-      (reference "VL53L1X1") (unit 1) (value "ToF distance sensor") (footprint "")
+      (reference "VL53L1X1") (unit 1) (value "ToF distance sensor") (footprint "Connector_PinHeader_2.54mm:PinHeader_1x06_P2.54mm_Horizontal")
     )
     (path "/05fe333d-6d2f-468a-bb69-555c38e6e071"
-      (reference "VL53L1X2") (unit 1) (value "ToF distance sensor") (footprint "")
+      (reference "VL53L1X2") (unit 1) (value "ToF distance sensor") (footprint "Connector_PinHeader_2.54mm:PinHeader_1x06_P2.54mm_Horizontal")
     )
     (path "/04817d1b-8dfa-4967-951b-473a12a01ac5"
-      (reference "VL53L1X3") (unit 1) (value "ToF distance sensor") (footprint "")
+      (reference "VL53L1X3") (unit 1) (value "ToF distance sensor") (footprint "Connector_PinHeader_2.54mm:PinHeader_1x06_P2.54mm_Horizontal")
     )
     (path "/8f221a57-1147-4b53-8a2c-091c1b87ae10"
-      (reference "VL53L1X4") (unit 1) (value "ToF distance sensor") (footprint "")
+      (reference "VL53L1X4") (unit 1) (value "ToF distance sensor") (footprint "Connector_PinHeader_2.54mm:PinHeader_1x06_P2.54mm_Horizontal")
     )
     (path "/d5ed175d-c824-4dc8-893c-bd149834d53f"
-      (reference "VL53L1X5") (unit 1) (value "ToF distance sensor") (footprint "")
-    )
-  )
+      (reference "VL53L1X5") (unit 1) (value "ToF distance sensor") (footprint "Connector_PinHeader_2.54mm:PinHeader_1x06_P2.54mm_Horizontal")
+    )
+  )
